Commit message: corrected length

File: xarm.URDF (robot description, URDF)
Before this commit: robot custom_robot, 6 links, 5 joints
Joints:
- joint joint5: origin xyz=0 0 4 -> xyz=0 0 14

Commit message: removed boxes from urdf

File: xarm.URDF (robot description, URDF)
Before this commit: robot custom_robot, 6 links, 5 joints
Links:
- link base_link: geometry 
- link link1: geometry 
- link link2: geometry 
- link link3: geometry 
- link link4: geometry 
- link link5: geometry 
Joints:
- joint joint1: origin xyz=0 0 5.5 -> xyz=0 0 0.055
- joint joint2: origin xyz=0 0 2 -> xyz=0 0 0.02
- joint joint3: origin xyz=0 0 10 -> xyz=0 0 0.10
- joint joint4: origin xyz=0 0 9.5 -> xyz=0 0 0.095
- joint joint5: origin xyz=0 0 14 -> xyz=0 0 0.014

Commit message: .

File: xarm.URDF (robot description, URDF)
Before this commit: robot custom_robot, 6 links, 5 joints
Links:
- removed link link5
Joints:
- removed joint joint5
- joint joint1: limit lower=-1.5707 upper=1.5707 effort=30 velocity=1.0 -> lower=-1.5707 upper=1.5707
- joint joint2: axis 1 0 0 -> 0 0 1; limit lower=-1.5707 upper=1.5707 effort=30 velocity=1.0 -> lower=-1.5707 upper=1.5707; origin xyz=0 0 0.02 -> xyz=0 0 0.02 rpy=-1.57 0 -1.57
- joint joint3: axis 1 0 0 -> 0 0 1; limit lower=-1.5707 upper=1.5707 effort=30 velocity=1.0 -> lower=-1.5707 upper=1.5707; origin xyz=0 0 0.10 -> xyz=0.10 0 0 rpy=-3.1415 0 0
- joint joint4: axis 1 0 0 -> 0 0 1; limit lower=-1.5707 upper=1.5707 effort=30 velocity=1.0 -> lower=-1.5707 upper=1.5707; origin xyz=0 0 0.095 -> xyz=0.095 0 0 rpy=-3.1415 0 0

File: xarm_large.URDF (robot description, URDF)
Before this commit: robot xArm, 7 links, 6 joints
Links:
- removed link link5
- removed link world
- link link1: geometry 
- link link2: geometry 
- link link3: geometry 
- link link4: geometry 
Joints:
- removed joint arm1
- removed joint arm2
- removed joint arm3
- removed joint arm4
- removed joint arm5
- removed joint world_joint
- added joint base_joint: type fixed, parent base_link, child link1, origin xyz=0 0 0 rpy=0 0 0
- added joint joint1: type continuous, parent link1, child link2, origin xyz=0.5 0.3 0 rpy=0 0 0, axis -0.9 0.15 0
- added joint joint2: type continuous, parent link1, child link3, origin xyz=-0.2 0.5 0 rpy=0 0 1.57, axis -1 0 0
- added joint joint3: type continuous, parent link3, child link4, origin xyz=0.5 0 0 rpy=0 0 -1.57, axis 0.707 -0.707 0

Commit message: added limits and corrected errors

File: xarm.URDF (robot description, URDF)
Before this commit: robot custom_robot, 5 links, 4 joints
Joints:
- joint joint1: limit lower=-1.5707 upper=1.5707 -> lower=-1.5707 upper=1.5707 effort=30 velocity=1.0
- joint joint2: limit lower=-1.5707 upper=1.5707 -> lower=-1.5707 upper=1.5707 effort=30 velocity=1.0
- joint joint3: limit lower=-1.5707 upper=1.5707 -> lower=-1.5707 upper=1.5707 effort=30 velocity=1.0
- joint joint4: limit lower=-1.5707 upper=1.5707 -> lower=-1.5707 upper=1.5707 effort=30 velocity=1.0

Commit message: finally working code

File: xarm.URDF (robot description, URDF)
Before this commit: robot custom_robot, 5 links, 4 joints
Links:
- removed link link1
- added link link5
- added link link6
Joints:
- removed joint joint1
- removed joint joint2
- added joint fixed_joint_2: type fixed, parent link3, child link2, origin xyz=-0.14 0 0 rpy=0 0 0
- added joint joint5: type revolute, parent link6, child link5, origin xyz=0 0 0.02 rpy=-1.57 0 0, axis 0 0 1, limit lower=-1.5707 upper=1.5707 effort=30 velocity=1.0
- added joint joint6: type revolute, parent base_link, child link6, origin xyz=0 0 0.055, axis 0 0 1, limit lower=-1.5707 upper=1.5707 effort=30 velocity=1.0
- joint joint3: origin xyz=0.10 0 0 rpy=-3.1415 0 0 -> xyz=-0.095 0 0 rpy=3.1415 0 0; parent link2 -> link4
- joint joint4: origin xyz=0.095 0 0 rpy=-3.1415 0 0 -> xyz=0 -0.1 0 rpy=3.1415 0 1.5707; parent link3 -> link5
